File: solenoid/solenoid.kicad_pcb (KiCad board)
At the start: 2 copper layers, 132 x 79 mm, 52 parts, among them J1 Arduino, J2 Arduino, J3 Conn_01x01_Male, J4 Conn_01x01_Male, Q1 TIP120, Q10 TIP120, Q11 TIP120, Q12 TIP120, Q13 TIP120, Q14 TIP120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

Commit message: mass production version updates
Parts:
- added J5: Conn_01x01, MountingHole:MountingHole_2.2mm_M2_Pad_Via, F.Cu at (84.3, 54.7)
- added J6: Conn_01x01, MountingHole:MountingHole_2.2mm_M2_Pad_Via, F.Cu at (74.5, 114.5)
- added J7: Conn_01x01, MountingHole:MountingHole_2.2mm_M2_Pad_Via, F.Cu at (198.0, 44.0)
- added J8: Conn_01x01, MountingHole:MountingHole_2.2mm_M2_Pad_Via, F.Cu at (197.5, 114.5)
- moved J4 9.03 mm to (84.0, 116.0)
- moved J3 1.79 mm to (80.5, 116.0)
Routing:
- net +12V: track 248.5 -> 253.3 mm
- net Earth: track 312.4 -> 315.0 mm
- net D16: track 154.5 -> 153.7 mm
Other:
- board text added: "Live loom solenoid driver v1.0 OSH"
