File: solenoid/solenoid.sch (KiCad schematic (older format))
At the start: 52 parts, among them J1 Arduino, J2 Arduino, J3 Conn_01x01_Male, J4 Conn_01x01_Male, Q1 TIP120, Q10 TIP120, Q11 TIP120, Q12 TIP120, Q13 TIP120, Q14 TIP120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

Commit message: mass production version updates
Parts:
- added J5, J6, J7, J8: Conn_01x01, MountingHole:MountingHole_2.2mm_M2_Pad_Via, symbol Connector_Generic:Conn_01x01
Changed lines of the file:
@@
 	0    -1   -1   0
 $EndComp
+$Comp
+L Connector_Generic:Conn_01x01 J5
+U 1 1 60F9D346
+P 8400 1350
+F 0 "J5" H 8480 1392 50  0000 L CNN
+F 1 "Conn_01x01" H 8480 1301 50  0000 L CNN
+F 2 "MountingHole:MountingHole_2.2mm_M2_Pad_Via" H 8400 1350 50  0001 C CNN
+F 3 "~" H 8400 1350 50  0001 C CNN
+	1    8400 1350
+	1    0    0    -1
+$EndComp
+$Comp
+L Connector_Generic:Conn_01x01 J6
+U 1 1 60FA3FF9
+P 8400 1550
+F 0 "J6" H 8480 1592 50  0000 L CNN
+F 1 "Conn_01x01" H 8480 1501 50  0000 L CNN
+F 2 "MountingHole:MountingHole_2.2mm_M2_Pad_Via" H 8400 1550 50  0001 C CNN
+F 3 "~" H 8400 1550 50  0001 C CNN
+	1    8400 1550
+	1    0    0    -1
+$EndComp
+$Comp
+L Connector_Generic:Conn_01x01 J7
+U 1 1 60FA6870
+P 8400 1750
+F 0 "J7" H 8480 1792 50  0000 L CNN
+F 1 "Conn_01x01" H 8480 1701 50  0000 L CNN
+F 2 "MountingHole:MountingHole_2.2mm_M2_Pad_Via" H 8400 1750 50  0001 C CNN
+F 3 "~" H 8400 1750 50  0001 C CNN
+	1    8400 1750
+	1    0    0    -1
+$EndComp
+$Comp
+L Connector_Generic:Conn_01x01 J8
+U 1 1 60FA792E
+P 8400 1950
+F 0 "J8" H 8480 1992 50  0000 L CNN
+F 1 "Conn_01x01" H 8480 1901 50  0000 L CNN
+F 2 "MountingHole:MountingHole_2.2mm_M2_Pad_Via" H 8400 1950 50  0001 C CNN
+F 3 "~" H 8400 1950 50  0001 C CNN
+	1    8400 1950
+	1    0    0    -1
+$EndComp
 $EndSCHEMATC
